Commit message: fix: visual and collision mismatch

File: IsaacGymEnvs/assets/urdf/hanu_a3_description/urdf/hanu_a3.urdf (robot description, URDF)
Before this commit: robot hanu_a3, 37 links, 36 joints
Links:
- link l_contact_sensor_1: mass 0.0027744190122019835 -> 0.05
- link r_contact_sensor_1: mass 0.0027744190122019835 -> 0.05
